Commit message: added inertia

File: src/fair_robot_description/urdf/robot.xacro (robot description, xacro)
@@ -2,4 +2,22 @@
 <robot xmlns:xacro="https://wiki.ros.org/xacro" name="robot">
 <xacro:property name="pi" value="3.14159265359" />
+    <xacro:macro name="inertial_box" params="mass x y z *origin">
+        <inertial>
+            <xacro:insert_block name="origin"/>
+            <mass value="${mass}" />
+            <inertia ixx="${(1/12) * mass * (y*y + z*z)}" ixy="0.0" ixz="0.0"
+                    iyy="${(1/12) * mass * (x*x + z*z)}" iyz="0.0"
+                    izz="${(1/12) * mass * (x*x + y*y)}" />
+        </inertial>
+    </xacro:macro>
+    <xacro:macro name="inertial_cylinder" params="mass length radius *origin">
+        <inertial>
+            <xacro:insert_block name="origin"/>
+            <mass value="${mass}" />
+            <inertia ixx="${(1/12) * mass * (3*radius*radius + length*length)}" ixy="0.0" ixz="0.0"
+                    iyy="${(1/12) * mass * (3*radius*radius + length*length)}" iyz="0.0"
+                    izz="${(1/2) * mass * (radius*radius)}" />
+        </inertial>
+    </xacro:macro>
     <!-- Materials -->
     <material name="white">
@@ -31,4 +49,7 @@
             </geometry>
         </collision>
+        <xacro:inertial_box mass="700" x="2.74" y="1.06" z="1.785">
+            <origin xyz="0 0 0" rpy="0 0 0"/>
+        </xacro:inertial_box>
     </link>
     <!-- Front Left Wheel -->
@@ -53,4 +74,7 @@
             </geometry>
         </collision>
+        <xacro:inertial_cylinder mass="15" length="0.15" radius="0.25">
+            <origin xyz="0 0 0" rpy="0 0 0"/>
+        </xacro:inertial_cylinder>
     </link>
     <!-- Front Right Wheel -->
@@ -75,4 +99,7 @@
             </geometry>
         </collision>
+        <xacro:inertial_cylinder mass="15" length="0.15" radius="0.25">
+            <origin xyz="0 0 0" rpy="0 0 0"/>
+        </xacro:inertial_cylinder>
     </link>
     <!-- Rear Left Wheel -->
@@ -97,4 +124,7 @@
             </geometry>
         </collision>
+        <xacro:inertial_cylinder mass="15" length="0.15" radius="0.25">
+            <origin xyz="0 0 0" rpy="0 0 0"/>
+        </xacro:inertial_cylinder>
     </link>
     <!-- Rear Right Wheel -->
@@ -119,4 +149,7 @@
             </geometry>
         </collision>
+        <xacro:inertial_cylinder mass="15" length="0.15" radius="0.25">
+            <origin xyz="0 0 0" rpy="0 0 0"/>
+        </xacro:inertial_cylinder>
     </link>
 </robot>
